File: pcb/brewBuddy.brd (EAGLE design)
At the start: 45.7 x 86.4 mm, 3 parts

Commit message: added Eagle files
Parts:
- moved 2.2TFT 3.81 mm to (20.3, 81.3)
Routing:
- net N$13: track 151.8 -> 148.0 mm
- net N$12: track 116.9 -> 120.7 mm
- net N$9: track 81.8 -> 78.3 mm
- net N$11: track 67.9 -> 65.9 mm
- net N$10: track 62.9 -> 64.5 mm
- net N$4: track 142.4 -> 141.8 mm
Changed lines of the file:
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@@
 </autorouter>
 <elements>
-<element name="2.2TFT" library="Adafruit_2.2_SPI_240x320" package="MICROBUILDER_1X10_ROUND_2MM" value="" x="16.51" y="81.28" rot="R180"/>
+<element name="2.2TFT" library="Adafruit_2.2_SPI_240x320" package="MICROBUILDER_1X10_ROUND_2MM" value="" x="20.32" y="81.28" rot="R180"/>
 <element name="U$1" library="Spark" package="PHOTON" value="PHOTON_WITH_HEADERS" x="34.29" y="38.1" rot="R180"/>
 <element name="MAX31855K" library="SparkFun_Thermocouple_Breakout" package="1X06_LONGPADS" value="6 Pad" x="6.35" y="66.04" rot="R270"/>
@@
 <wire x1="6.35" y1="60.96" x2="1.27" y2="60.96" width="0.4064" layer="1"/>
 <wire x1="1.27" y1="60.96" x2="1.27" y2="77.47" width="0.4064" layer="1"/>
-<wire x1="1.27" y1="77.47" x2="10.51" y2="77.47" width="0.4064" layer="1"/>
-<wire x1="10.51" y1="77.47" x2="10.51" y2="81.28" width="0.4064" layer="1"/>
-<wire x1="10.51" y1="81.28" x2="10.16" y2="81.28" width="0.4064" layer="1"/>
+<wire x1="1.27" y1="77.47" x2="9.875" y2="77.47" width="0.4064" layer="1"/>
+<wire x1="9.875" y1="77.47" x2="9.84" y2="81.28" width="0.4064" layer="1"/>
+<wire x1="9.84" y1="81.28" x2="10.16" y2="81.28" width="0.4064" layer="1"/>
 <wire x1="10.16" y1="81.28" x2="10.16" y2="83.82" width="0.4064" layer="1"/>
 <wire x1="10.16" y1="83.82" x2="44.45" y2="83.82" width="0.4064" layer="1"/>
@@
 <contactref element="2.2TFT" pad="8"/>
 <contactref element="MAX31855K" pad="4"/>
-<wire x1="12.51" y1="81.28" x2="12.7" y2="81.28" width="0.4064" layer="16"/>
+<wire x1="12.4" y1="81.28" x2="12.7" y2="81.28" width="0.4064" layer="16"/>
 <wire x1="12.7" y1="81.28" x2="12.7" y2="58.42" width="0.4064" layer="16"/>
 <wire x1="12.7" y1="58.42" x2="6.35" y2="58.42" width="0.4064" layer="16"/>
-<wire x1="12.51" y1="81.28" x2="12.7" y2="81.28" width="0.4064" layer="1"/>
+<wire x1="12.4" y1="81.28" x2="12.7" y2="81.28" width="0.4064" layer="1"/>
 <wire x1="12.7" y1="81.28" x2="12.7" y2="44.45" width="0.4064" layer="1"/>
 <wire x1="12.7" y1="44.45" x2="36.83" y2="44.45" width="0.4064" layer="1"/>
@@
 <via x="39.37" y="53.34" extent="1-16" drill="1"/>
 <wire x1="39.37" y1="53.34" x2="39.37" y2="76.2" width="0.4064" layer="1"/>
-<wire x1="39.37" y1="76.2" x2="16.51" y2="76.2" width="0.4064" layer="1"/>
-<wire x1="16.51" y1="76.2" x2="16.51" y2="81.28" width="0.4064" layer="1"/>
+<wire x1="39.37" y1="76.2" x2="19.05" y2="77.47" width="0.4064" layer="1"/>
+<wire x1="19.05" y1="77.47" x2="17.52" y2="81.28" width="0.4064" layer="1"/>
 </signal>
 <signal name="N$10">
@@
 <via x="33.02" y="53.34" extent="1-16" drill="1"/>
 <wire x1="33.02" y1="53.34" x2="33.02" y2="71.12" width="0.4064" layer="1"/>
-<wire x1="33.02" y1="71.12" x2="20.32" y2="71.12" width="0.4064" layer="1"/>
-<via x="20.32" y="71.12" extent="1-16" drill="1"/>
-<wire x1="20.32" y1="71.12" x2="20.51" y2="73.66" width="0.4064" layer="16"/>
-<wire x1="20.51" y1="73.66" x2="20.51" y2="81.28" width="0.4064" layer="16"/>
+<wire x1="33.02" y1="71.12" x2="22.86" y2="71.12" width="0.4064" layer="1"/>
+<via x="22.86" y="71.12" extent="1-16" drill="1"/>
+<wire x1="22.86" y1="71.12" x2="19.24" y2="71.12" width="0.4064" layer="16"/>
+<wire x1="19.24" y1="71.12" x2="22.66" y2="81.28" width="0.4064" layer="16"/>
 </signal>
 <signal name="N$11">
@@
 <via x="36.195" y="53.34" extent="1-16" drill="1"/>
 <wire x1="36.195" y1="53.34" x2="36.195" y2="73.66" width="0.4064" layer="1"/>
-<wire x1="36.195" y1="73.66" x2="22.86" y2="73.66" width="0.4064" layer="1"/>
-<via x="22.86" y="73.66" extent="1-16" drill="1"/>
-<wire x1="22.86" y1="73.66" x2="22.51" y2="74.93" width="0.4064" layer="16"/>
-<wire x1="22.51" y1="74.93" x2="22.51" y2="81.28" width="0.4064" layer="16"/>
+<wire x1="36.195" y1="73.66" x2="25.4" y2="73.66" width="0.4064" layer="1"/>
+<via x="25.4" y="73.66" extent="1-16" drill="1"/>
+<wire x1="25.4" y1="73.66" x2="23.78" y2="77.47" width="0.4064" layer="16"/>
+<wire x1="23.78" y1="77.47" x2="25.2" y2="81.28" width="0.4064" layer="16"/>
 </signal>
 <signal name="N$12">
 <contactref element="2.2TFT" pad="2"/>
 <contactref element="U$1" pad="24"/>
-<wire x1="24.51" y1="81.28" x2="24.13" y2="83.82" width="0.4064" layer="16"/>
-<wire x1="24.13" y1="83.82" x2="1.27" y2="83.82" width="0.4064" layer="16"/>
+<wire x1="27.76" y1="81.28" x2="27.94" y2="83.82" width="0.4064" layer="16"/>
+<wire x1="27.94" y1="83.82" x2="1.27" y2="83.82" width="0.4064" layer="16"/>
 <wire x1="1.27" y1="83.82" x2="1.27" y2="6.35" width="0.4064" layer="16"/>
 <wire x1="1.27" y1="6.35" x2="6.35" y2="6.35" width="0.4064" layer="16"/>
@@
 <contactref element="2.2TFT" pad="1"/>
 <contactref element="U$1" pad="21"/>
-<wire x1="26.51" y1="81.28" x2="26.67" y2="77.47" width="0.4064" layer="16"/>
-<wire x1="26.67" y1="77.47" x2="43.18" y2="77.47" width="0.4064" layer="16"/>
+<wire x1="30.32" y1="81.28" x2="30.48" y2="77.47" width="0.4064" layer="16"/>
+<wire x1="30.48" y1="77.47" x2="43.18" y2="77.47" width="0.4064" layer="16"/>
 <wire x1="43.18" y1="77.47" x2="43.18" y2="0" width="0.4064" layer="16"/>
 <wire x1="43.18" y1="0" x2="8.89" y2="0" width="0.4064" layer="16"/>
@@
 <contactref element="U$1" pad="7"/>
 <contactref element="MAX31855K" pad="5"/>
-<wire x1="14.51" y1="81.28" x2="13.97" y2="81.28" width="0.4064" layer="16"/>
+<wire x1="14.96" y1="81.28" x2="13.97" y2="81.28" width="0.4064" layer="16"/>
 <wire x1="13.97" y1="81.28" x2="13.97" y2="55.88" width="0.4064" layer="16"/>
 <wire x1="13.97" y1="55.88" x2="6.35" y2="55.88" width="0.4064" layer="16"/>
